File: Audio.sch (KiCad schematic (older format))
At the start: 0 parts

Commit message: got the schematic done
Parts:
- added C? (x2): CAP, symbol pspice:CAP
- added J?: 3.5mmStereoJack, symbol NewSymbols:3.5mmStereoJack
- added J?: Conn_01x02_Male, symbol Connector:Conn_01x02_Male
- added J?: DB25_Female_MountingHoles, symbol Connector:DB25_Female_MountingHoles
- added R? (x4): R, symbol Device:R
Connections:
- net ASignal1: now also J?.24 (P24)
- net ASignal2: now also J?.10
- net ASignal3: now also J?.21 (P21)
- net ASignal4: now also J?.7
- net ASignal5: now also J?.18 (P18)
- net ASignal6: now also J?.4
- net ASignal7: now also J?.15 (P15)
- net ASignal8: now also J?.1
- new net GND: J?.1 (GND), J?.11, J?.16 (P16), J?.19 (P19), J?.2, J?.22 (P22), J?.25 (P25), J?.5, J?.8, R?.2, R?.2
- new net OPAMP1_VINM: C?.2, R?.1, R?.2
- new net OPAMP1_VOUT: C?.1, J?.2 (Pin_2), J?.4 (ExtraRightChannel), J?.5 (RightChannel), R?.1
- new net OPAMP2_VINM: C?.2, R?.1, R?.2
- new net OPAMP2_VOUT: C?.1, J?.1 (Pin_1), J?.2 (LeftChannel), J?.3 (ExtraLeftChannel), R?.1

Commit message: added the needed footprints
Parts:
- C11, C12: renamed from C?; footprint (none) -> Capacitor_THT:CP_Radial_D8.0mm_P3.50mm
- J10: renamed from J?; footprint (none) -> Connector_Dsub:DSUB-25_Female_Horizontal_P2.77x2.84mm_EdgePinOffset7.70mm_Housed_MountingHolesOffset9.12mm
- J11: renamed from J?; footprint (none) -> Connector_PinHeader_2.54mm:PinHeader_1x02_P2.54mm_Vertical
- J12: renamed from J?; footprint (none) -> LocalFootPrints:3.5mmAudioJack
- R10, R11, R8, R9: renamed from R?; footprint (none) -> Resistor_THT:R_Axial_DIN0207_L6.3mm_D2.5mm_P7.62mm_Horizontal
Changed lines of the file:
@@
 $EndSheet
 $Comp
-L Connector:Conn_01x02_Male J?
+L Connector:Conn_01x02_Male J11
 U 1 1 5FC29CDB
 P 3050 6300
-F 0 "J?" H 3158 6481 50  0000 C CNN
+F 0 "J11" H 3158 6481 50  0000 C CNN
 F 1 "Conn_01x02_Male" H 3158 6390 50  0000 C CNN
-F 2 "" H 3050 6300 50  0001 C CNN
+F 2 "Connector_PinHeader_2.54mm:PinHeader_1x02_P2.54mm_Vertical" H 3050 6300 50  0001 C CNN
 F 3 "~" H 3050 6300 50  0001 C CNN
 	1    3050 6300
@@
 Connection ~ 3250 6000
 $Comp
-L Connector:DB25_Female_MountingHoles J?
+L Connector:DB25_Female_MountingHoles J10
 U 1 1 5FC31E52
 P 2650 2450
-F 0 "J?" H 2830 2452 50  0000 L CNN
+F 0 "J10" H 2830 2452 50  0000 L CNN
 F 1 "DB25_Female_MountingHoles" H 2830 2361 50  0000 L CNN
-F 2 "" H 2650 2450 50  0001 C CNN
+F 2 "Connector_Dsub:DSUB-25_Female_Horizontal_P2.77x2.84mm_EdgePinOffset7.70mm_Housed_MountingHolesOffset9.12mm" H 2650 2450 50  0001 C CNN
 F 3 " ~" H 2650 2450 50  0001 C CNN
 	1    2650 2450
@@
 OPAMP2_VINM
 $Comp
-L power:GND #PWR?
+L power:GND #PWR023
 U 1 1 5FBDD330
 P 1450 7150
-F 0 "#PWR?" H 1450 6900 50  0001 C CNN
+F 0 "#PWR023" H 1450 6900 50  0001 C CNN
 F 1 "GND" V 1455 7022 50  0000 R CNN
 F 2 "" H 1450 7150 50  0001 C CNN
@@
 $EndComp
 $Comp
-L Device:R R?
+L Device:R R9
 U 1 1 5FBDE2E1
 P 1600 7150
-F 0 "R?" V 1393 7150 50  0000 C CNN
+F 0 "R9" V 1393 7150 50  0000 C CNN
 F 1 "R" V 1484 7150 50  0000 C CNN
-F 2 "" V 1530 7150 50  0001 C CNN
+F 2 "Resistor_THT:R_Axial_DIN0207_L6.3mm_D2.5mm_P7.62mm_Horizontal" V 1530 7150 50  0001 C CNN
 F 3 "~" H 1600 7150 50  0001 C CNN
 	1    1600 7150
@@
 	2900 6450 3250 6450
 $Comp
-L pspice:CAP C?
+L pspice:CAP C12
 U 1 1 5FBE0FA7
 P 2450 7600
-F 0 "C?" V 2135 7600 50  0000 C CNN
+F 0 "C12" V 2135 7600 50  0000 C CNN
 F 1 "CAP" V 2226 7600 50  0000 C CNN
-F 2 "" H 2450 7600 50  0001 C CNN
+F 2 "Capacitor_THT:CP_Radial_D8.0mm_P3.50mm" H 2450 7600 50  0001 C CNN
 F 3 "~" H 2450 7600 50  0001 C CNN
 	1    2450 7600
@@
 $EndComp
 $Comp
-L Device:R R?
+L Device:R R11
 U 1 1 5FBE3EA0
 P 2450 7150
-F 0 "R?" V 2243 7150 50  0000 C CNN
+F 0 "R11" V 2243 7150 50  0000 C CNN
 F 1 "R" V 2334 7150 50  0000 C CNN
-F 2 "" V 2380 7150 50  0001 C CNN
+F 2 "Resistor_THT:R_Axial_DIN0207_L6.3mm_D2.5mm_P7.62mm_Horizontal" V 2380 7150 50  0001 C CNN
 F 3 "~" H 2450 7150 50  0001 C CNN
 	1    2450 7150
@@
 	1750 7150 1950 7150
 $Comp
-L power:GND #PWR?
+L power:GND #PWR022
 U 1 1 5FBE66DF
 P 1400 5350
-F 0 "#PWR?" H 1400 5100 50  0001 C CNN
+F 0 "#PWR022" H 1400 5100 50  0001 C CNN
 F 1 "GND" V 1405 5222 50  0000 R CNN
 F 2 "" H 1400 5350 50  0001 C CNN
@@
 $EndComp
 $Comp
-L Device:R R?
+L Device:R R8
 U 1 1 5FBE6C5B
 P 1550 5350
-F 0 "R?" V 1343 5350 50  0000 C CNN
+F 0 "R8" V 1343 5350 50  0000 C CNN
 F 1 "R" V 1434 5350 50  0000 C CNN
-F 2 "" V 1480 5350 50  0001 C CNN
+F 2 "Resistor_THT:R_Axial_DIN0207_L6.3mm_D2.5mm_P7.62mm_Horizontal" V 1480 5350 50  0001 C CNN
 F 3 "~" H 1550 5350 50  0001 C CNN
 	1    1550 5350
@@
 	1950 5350 1950 5700
 $Comp
-L Device:R R?
+L Device:R R10
 U 1 1 5FBE7A9B
 P 2400 5350
-F 0 "R?" V 2193 5350 50  0000 C CNN
+F 0 "R10" V 2193 5350 50  0000 C CNN
 F 1 "R" V 2284 5350 50  0000 C CNN
-F 2 "" V 2330 5350 50  0001 C CNN
+F 2 "Resistor_THT:R_Axial_DIN0207_L6.3mm_D2.5mm_P7.62mm_Horizontal" V 2330 5350 50  0001 C CNN
 F 3 "~" H 2400 5350 50  0001 C CNN
 	1    2400 5350
@@
 	2900 6000 3250 6000
 $Comp
-L pspice:CAP C?
+L pspice:CAP C11
 U 1 1 5FBEBFAA
 P 2400 4950
-F 0 "C?" V 2085 4950 50  0000 C CNN
+F 0 "C11" V 2085 4950 50  0000 C CNN
 F 1 "CAP" V 2176 4950 50  0000 C CNN
-F 2 "" H 2400 4950 50  0001 C CNN
+F 2 "Capacitor_THT:CP_Radial_D8.0mm_P3.50mm" H 2400 4950 50  0001 C CNN
 F 3 "~" H 2400 4950 50  0001 C CNN
 	1    2400 4950
@@
 	3250 6400 3650 6400
 $Comp
-L NewSymbols:3.5mmStereoJack J?
+L NewSymbols:3.5mmStereoJack J12
 U 1 1 5FC27E79
 P 4150 6200
-F 0 "J?" V 4079 6719 50  0000 L CNN
+F 0 "J12" V 4079 6719 50  0000 L CNN
 F 1 "3.5mmStereoJack" V 4170 6719 50  0000 L CNN
-F 2 "" H 4100 6800 50  0001 C CNN
+F 2 "LocalFootPrints:3.5mmAudioJack" H 4100 6800 50  0001 C CNN
 F 3 "" H 4100 6800 50  0001 C CNN
 	1    4150 6200
@@
 Connection ~ 3650 6400
 $Comp
-L power:GND #PWR?
+L power:GND #PWR032
 U 1 1 5FBEFC0D
 P 3650 5850
-F 0 "#PWR?" H 3650 5600 50  0001 C CNN
+F 0 "#PWR032" H 3650 5600 50  0001 C CNN
 F 1 "GND" V 3655 5722 50  0000 R CNN
 F 2 "" H 3650 5850 50  0001 C CNN
@@
 $EndComp
 $Comp
-L power:GND #PWR?
+L power:GND #PWR024
 U 1 1 5FBF03ED
 P 2950 1350
-F 0 "#PWR?" H 2950 1100 50  0001 C CNN
+F 0 "#PWR024" H 2950 1100 50  0001 C CNN
 F 1 "GND" V 2955 1222 50  0000 R CNN
 F 2 "" H 2950 1350 50  0001 C CNN
@@
 $EndComp
 $Comp
-L power:GND #PWR?
+L power:GND #PWR025
 U 1 1 5FBF09BD
 P 2950 1650
-F 0 "#PWR?" H 2950 1400 50  0001 C CNN
+F 0 "#PWR025" H 2950 1400 50  0001 C CNN
 F 1 "GND" V 2955 1522 50  0000 R CNN
 F 2 "" H 2950 1650 50  0001 C CNN
@@
 $EndComp
 $Comp
-L power:GND #PWR?
+L power:GND #PWR026
 U 1 1 5FBF1F67
 P 2950 1950
-F 0 "#PWR?" H 2950 1700 50  0001 C CNN
+F 0 "#PWR026" H 2950 1700 50  0001 C CNN
 F 1 "GND" V 2955 1822 50  0000 R CNN
 F 2 "" H 2950 1950 50  0001 C CNN
@@
 $EndComp
 $Comp
-L power:GND #PWR?
+L power:GND #PWR027
 U 1 1 5FBF32A1
 P 2950 2250
-F 0 "#PWR?" H 2950 2000 50  0001 C CNN
+F 0 "#PWR027" H 2950 2000 50  0001 C CNN
 F 1 "GND" V 2955 2122 50  0000 R CNN
 F 2 "" H 2950 2250 50  0001 C CNN
@@
 $EndComp
 $Comp
-L power:GND #PWR?
+L power:GND #PWR028
 U 1 1 5FBF408D
 P 2950 2550
-F 0 "#PWR?" H 2950 2300 50  0001 C CNN
+F 0 "#PWR028" H 2950 2300 50  0001 C CNN
 F 1 "GND" V 2955 2422 50  0000 R CNN
 F 2 "" H 2950 2550 50  0001 C CNN
@@
 $EndComp
 $Comp
-L power:GND #PWR?
+L power:GND #PWR029
 U 1 1 5FBF4B1B
 P 2950 2850
-F 0 "#PWR?" H 2950 2600 50  0001 C CNN
+F 0 "#PWR029" H 2950 2600 50  0001 C CNN
 F 1 "GND" V 2955 2722 50  0000 R CNN
 F 2 "" H 2950 2850 50  0001 C CNN
@@
 $EndComp
 $Comp
-L power:GND #PWR?
+L power:GND #PWR030
 U 1 1 5FBF5695
 P 2950 3150
-F 0 "#PWR?" H 2950 2900 50  0001 C CNN
+F 0 "#PWR030" H 2950 2900 50  0001 C CNN
 F 1 "GND" V 2955 3022 50  0000 R CNN
 F 2 "" H 2950 3150 50  0001 C CNN
@@
 $EndComp
 $Comp
-L power:GND #PWR?
+L power:GND #PWR031
 U 1 1 5FBF5FE5
 P 2950 3450
-F 0 "#PWR?" H 2950 3200 50  0001 C CNN
+F 0 "#PWR031" H 2950 3200 50  0001 C CNN
 F 1 "GND" V 2955 3322 50  0000 R CNN
 F 2 "" H 2950 3450 50  0001 C CNN

Commit message: layout time
Parts:
- C11: footprint Capacitor_THT:CP_Radial_D8.0mm_P3.50mm -> Capacitor_THT:C_Radial_D10.0mm_H12.5mm_P5.00mm
- C12: footprint Capacitor_THT:CP_Radial_D8.0mm_P3.50mm -> Capacitor_THT:CP_Radial_D8.0mm_P5.00mm
Changed lines of the file:
@@
 F 0 "C12" V 2135 7600 50  0000 C CNN
 F 1 "CAP" V 2226 7600 50  0000 C CNN
-F 2 "Capacitor_THT:CP_Radial_D8.0mm_P3.50mm" H 2450 7600 50  0001 C CNN
+F 2 "Capacitor_THT:CP_Radial_D8.0mm_P5.00mm" H 2450 7600 50  0001 C CNN
 F 3 "~" H 2450 7600 50  0001 C CNN
 	1    2450 7600
@@
 F 0 "C11" V 2085 4950 50  0000 C CNN
 F 1 "CAP" V 2176 4950 50  0000 C CNN
-F 2 "Capacitor_THT:CP_Radial_D8.0mm_P3.50mm" H 2400 4950 50  0001 C CNN
+F 2 "Capacitor_THT:C_Radial_D10.0mm_H12.5mm_P5.00mm" H 2400 4950 50  0001 C CNN
 F 3 "~" H 2400 4950 50  0001 C CNN
 	1    2400 4950
