File: DevBoard.sch (KiCad schematic (older format))
At the start: 23 parts, among them J1 6.35mmMonoAudioJack, J2 6.35mmMonoAudioJack

Commit message: got the schematic done
Parts:
- removed J1, J2: 6.35mmMonoAudioJack, LocalFootPrints:6.35mmMonoAudioJack, symbol NewSymbols:6.35mmMonoAudioJack
- added J?: DIN-5_180degree, symbol Connector:DIN-5_180degree
- added J?: Debug Headers, symbol Connector_Generic:Conn_02x04_Odd_Even
- added R? (x2): R 220, symbol Device:R
Connections:
- net Audio/ASignal6: now also U?.16 (PA2); no longer U?.15 (PA1)
- net Audio/ASignal7: now also U?.20 (PA4); no longer U?.16 (PA2)
- net Audio/ASignal8: now also U?.21 (PA5); no longer U?.17 (PA3)
- net Audio/ASignal9: now also U?.22 (PA6)
- net GND: now also J?.2, J?.2 (Pin_2)
- net DebugPort3: now reaches U?.2 (PC13)
- net DebugPort3: now also J?.7 (Pin_7)
- net Audio/OPAMP2_VINM: now reaches U?.23 (PA7)
- net ASignal10: now reaches U?.24 (PC4)
- net OPAMP2_VOUT: now reaches U?.26 (PB0)
- net Keyboard_DATA: now reaches U?.29 (PB10)
- net DebugPort4: now reaches U?.3 (PC14)
- net DebugPort4: now also J?.8 (Pin_8)
- net Keyboard_CLK: now reaches U?.33 (PB12)
- net PS2_SCK: now reaches U?.34 (PB13)
- net PS2_MISO: now reaches U?.35 (PB14)
- net PS2_MOSI: now reaches U?.36 (PB15)
- net DebugUartTX: now reaches U?.51 (PC10)
- net DebugUartTX: now also J?.3 (Pin_3)
- net DebugUartRX: now reaches U?.52 (PC11)
- net DebugUartRX: now also J?.4 (Pin_4)
- net MIDI_UART: now reaches U?.53 (PC12)
- net MIDI_UART: now also R?.1
- net PS2_AWK: now reaches U?.58 (PB6)
- net DebugPort2: now reaches U?.59 (PB7)
- net DebugPort2: now also J?.6 (Pin_6)
- net DebugPort1: now reaches U?.61 (PB8)
- net DebugPort1: now also J?.5 (Pin_5)
- net PS2_CS: now reaches U?.62 (PB9)
- net G_5V: now reaches U?.3 (VIN)
- net G_5V: now also J?.1 (VBUS), R?.2
- net VCC_3_3 renamed G_3.3
- net G_3.3: now also J?.1 (Pin_1)
- new net: J?.4, R?.1
- new net: J?.5, R?.2
- new net Audio/OPAMP1_VINM: U?.15 (PA1)
- new net Audio/OPAMP1_VOUT: U?.17 (PA3)

Commit message: added the needed footprints
Parts:
- C1, C10, C2, C3, C4, C5, C6, C7, C8, C9: renamed from C?; footprint (none) -> Capacitor_SMD:C_0603_1608Metric
- D1: renamed from D?; footprint (none) -> LED_THT:LED_D5.0mm
- FB1: renamed from FB?; footprint (none) -> Inductor_SMD:L_0603_1608Metric
- J1: renamed from J?; footprint (none) -> Connector_PinHeader_2.54mm:PinHeader_1x06_P2.54mm_Vertical
- J2: renamed from J?; footprint (none) -> digikey-footprints:USB_Micro_B_Female_1050170001
- J3: renamed from J?; footprint (none) -> Connector_PinHeader_2.54mm:PinHeader_2x04_P2.54mm_Vertical
- R1, R2, R4, R5: renamed from R?; footprint (none) -> Resistor_THT:R_Axial_DIN0207_L6.3mm_D2.5mm_P7.62mm_Horizontal
- R3: renamed from R?; value R -> R 100k; footprint (none) -> Resistor_THT:R_Axial_DIN0207_L6.3mm_D2.5mm_P7.62mm_Horizontal
- SW1: renamed from SW?; footprint (none) -> Button_Switch_Keyboard:SW_Cherry_MX_1.00u_PCB
- gave numbers to parts that had none: 4

Commit message: layout time
Parts:
- J4: value DIN-5_180degree -> MIDI_TX_Out; footprint (none) -> LocalFootPrints:DIN5_midi
Changed lines of the file:
@@
 P 9650 3550
 F 0 "J4" H 9650 3275 50  0000 C CNN
-F 1 "DIN-5_180degree" H 9650 3184 50  0000 C CNN
-F 2 "" H 9650 3550 50  0001 C CNN
+F 1 "MIDI_TX_Out" H 9650 3184 50  0000 C CNN
+F 2 "LocalFootPrints:DIN5_midi" H 9650 3550 50  0001 C CNN
 F 3 "http://www.mouser.com/ds/2/18/40_c091_abd_e-75918.pdf" H 9650 3550 50  0001 C CNN
 	1    9650 3550
